File: kicad/NEXUS-MacroPad.kicad_sch (KiCad schematic)
At the start: 16 parts, among them J1 OLED wires: GND VCC SCL SDA, SW1 MX 1u, SW2 MX 1u, SW3 MX 1u, SW4 MX 1u, SW5 MX 1u, SW6 MX 1u, U1 Orpheus Pico / Pico compatible

Commit message: Update public identity and project links
Other:
- company: Hrushi / NEXUS -> hirsu / NEXUS
